Commit message: updated with cost maps

File: youbot_description/robots/youbot.urdf.xacro (robot description, xacro)
@@ -22,4 +22,6 @@
   <!-- sensors -->
   <xacro:include filename="$(find youbot_description)/urdf/sensors/hokuyo_urg04_laser.urdf.xacro"/>
+  <!-- kinect -->
+  <xacro:include filename="$(find youbot_description)/urdf/sensors/kinect_camera.urdf.xacro"/>
   <!-- Now we can start using the macros xacro:included above to define the actual youbot -->
   <!-- The first use of a macro.  This one was defined in base.urdf.xacro above.
@@ -45,3 +47,7 @@
     <origin xyz="0.3 0 -0.03" rpy="0 0 0"/>
   </xacro:hokuyo_urg04_laser>
+  <!-- kinect camera front -->
+  <xacro:kinect_camera name="kinect_camera" parent="arm_link_4">
+    <origin xyz="0.2 0 0.33" rpy="0 0 0" />
+  </xacro:kinect_camera>
 </robot>

File: youbot_description/urdf/sensors/kinect_camera.gazebo.xacro (robot description, xacro)
@@ -41,5 +41,5 @@
       <controller:gazebo_ros_camera name="${name}_rgb_frame_controller" plugin="libgazebo_ros_camera.so">
         <alwaysOn>true</alwaysOn>
-        <updateRate>20.0</updateRate>
+        <updateRate>30.0</updateRate>
         <imageTopicName>/camera/rgb/image_raw</imageTopicName>
         <cameraInfoTopicName>/camera/rgb/camera_info</cameraInfoTopicName>

File: youbot_description/urdf/sensors/kinect_camera.urdf.xacro (robot description, xacro)
@@ -24,4 +24,5 @@
        <mesh filename="package://youbot_description/meshes/sensors/kinect.dae"/>
       </geometry>
+      <material name="orange" />
     </visual>
     <collision>
@@ -89,5 +90,5 @@
   </link>
   <!-- for simulation -->
-  <xacro:kinect_camera_gazebo name="openni" />
+  <xacro:kinect_camera_gazebo name="kinect"/>
 </xacro:macro>
 </root>

File: youbot_simulation/youbot_gazebo_worlds/urdf/robocup_at_work_2012.urdf (robot description, URDF)
Before this commit: robot arena, 10 links, 9 joints
Links:
- removed link wall_4
- removed link wall_5
- added link orange_box, mass 1e-2; collision box size=${2*0.15748} ${2*0.15748} ${0.35*0.8508}}; visual box size=${2*0.15748} ${2*0.15748} ${0.35*0.8508}
Joints:
- removed joint join3
- removed joint join4
- added joint join_box: type fixed, parent wall_8, child orange_box, origin xyz=${5*0.6} -0.15 0.0 rpy=0 0 0

Commit message: updates

File: youbot_description/robots/youbot.urdf.xacro (robot description, xacro)
@@ -24,4 +24,6 @@
   <!-- kinect -->
   <xacro:include filename="$(find youbot_description)/urdf/sensors/kinect_camera.urdf.xacro"/>
+  <!-- obstacle -->
+<!--   <xacro:include filename="$(find youbot_description)/urdf/youbot_obstacle/obstacle.urdf.xacro" /> -->
   <!-- Now we can start using the macros xacro:included above to define the actual youbot -->
   <!-- The first use of a macro.  This one was defined in base.urdf.xacro above.
@@ -47,4 +49,5 @@
     <origin xyz="0.3 0 -0.03" rpy="0 0 0"/>
   </xacro:hokuyo_urg04_laser>
+  <!-- <xacro:youbot_obstacle_box_gazebo/> -->
   <!-- kinect camera front -->
 <!--   <xacro:kinect_camera name="kinect_camera" parent="arm_link_4">

File: youbot_simulation/youbot_gazebo_worlds/urdf/robocup_at_work_2012.urdf (robot description, URDF)
Before this commit: robot arena, 9 links, 8 joints
Links:
- link orange_box: geometry collision box size=${2*0.15748} ${2*0.15748} ${0.35*0.8508}; visual box size=${2*0.15748} ${2*0.15748} ${0.35*0.8508}

Commit message: updating base_footprint position

File: youbot_description/robots/youbot.urdf.xacro (robot description, xacro)
@@ -5,7 +5,7 @@
        xmlns:xacro="http://playerstage.sourceforge.net/gazebo/xmlschema/#interface"
        name="youbot" >
+  <xacro:property name="offset" value="-3.8" />
   <!-- The following xacro:included files set up definitions of parts of the robot body -->
   <!-- misc common stuff? -->
-  <xacro:include filename="$(find youbot_description)/urdf/common.xacro" />
   <!-- youbot base -->
   <xacro:include filename="$(find youbot_description)/urdf/youbot_base/base.urdf.xacro" />
@@ -37,20 +37,20 @@
   <xacro:youbot_base name="base"/>
   <xacro:youbot_plate name="plate" parent="base_link">
-    <origin xyz="-0.159 0 0.046" rpy="0 0 0" />
+    <origin xyz="${-0.159} 0 0.046" rpy="0 0 0" />
   </xacro:youbot_plate>
   <xacro:youbot_arm name="arm" parent="base_link">
-    <origin xyz="0.143 0 0.046" rpy="0 0 0" />
+    <origin xyz="${0.143} 0 0.046" rpy="0 0 0" />
   </xacro:youbot_arm>
   <xacro:youbot_gripper name="gripper" parent="arm_link_5">
-    <origin xyz="0 0 0" rpy="0 0 0" />
+    <origin xyz="${0} 0 0" rpy="0 0 0" />
   </xacro:youbot_gripper>
   <!-- base laser front -->
   <xacro:hokuyo_urg04_laser name="base_laser_front" parent="base" ros_topic="scan" update_rate="10" min_angle="-1.57" max_angle="1.57">
-    <origin xyz="0.3 0 -0.03" rpy="0 0 0"/>
+    <origin xyz="${0.3} 0 -0.03" rpy="0 0 0"/>
   </xacro:hokuyo_urg04_laser>
   <!-- <xacro:youbot_obstacle_box_gazebo/> -->
   <!-- kinect camera front -->
-<!--   <xacro:kinect_camera name="kinect_camera" parent="arm_link_4">
-    <origin xyz="0.2 0 0.33" rpy="0 0 0" />
-  </xacro:kinect_camera> -->
+  <xacro:kinect_camera name="kinect_camera" parent="arm_link_4">
+    <origin xyz="${0.2} 0 0.33" rpy="0 0 0" />
+  </xacro:kinect_camera>
 </robot>

File: youbot_description/urdf/youbot_base/base.urdf.xacro (robot description, xacro)
@@ -32,4 +32,5 @@
   <property name="wheel_joint_velocity" value="10"/>
   <property name="wheel_joint_safety_k_velocity" value="10.0"/>
+  <property name="base_offset" value="-3.8" />
   <xacro:macro name="youbot_base" params="name">
     <link name="${name}_footprint">
@@ -54,5 +55,5 @@
     </link>
     <joint name="${name}_footprint_joint" type="fixed">
-      <origin xyz="0 0 0" rpy="0 0 0"/>
+      <origin xyz="${base_offset} 0 0" rpy="0 0 0"/>
       <child link="${name}_link"/>
       <parent link="${name}_footprint"/>

Commit message: added Jennifer Buehler's common-sensors as submodule

File: youbot_description/robots/youbot.urdf.xacro (robot description, xacro)
@@ -24,6 +24,5 @@
   <!-- kinect -->
   <xacro:include filename="$(find youbot_description)/urdf/sensors/kinect_camera.urdf.xacro"/>
-  <!-- obstacle -->
-<!--   <xacro:include filename="$(find youbot_description)/urdf/youbot_obstacle/obstacle.urdf.xacro" /> -->
+  <xacro:include filename="$(find common_sensors)/urdf/sensors/kinect2.urdf.xacro"/>
   <!-- Now we can start using the macros xacro:included above to define the actual youbot -->
   <!-- The first use of a macro.  This one was defined in base.urdf.xacro above.
@@ -49,8 +48,7 @@
     <origin xyz="${0.3} 0 -0.03" rpy="0 0 0"/>
   </xacro:hokuyo_urg04_laser>
-  <!-- <xacro:youbot_obstacle_box_gazebo/> -->
-  <!-- kinect camera front -->
-  <xacro:kinect_camera name="kinect_camera" parent="arm_link_4">
-    <origin xyz="${0.2} 0 0.33" rpy="0 0 0" />
-  </xacro:kinect_camera>
+  <!-- kinect2 camera from Jennifer Buehler -->
+  <xacro:kinect2 name="kinect_camera_rgb" parent="base_link" >
+    <origin xyz="${0.35} 0 0.25" rpy="0 0 0" />
+  </xacro:kinect2>
 </robot>

File: youbot_description/urdf/sensors/kinect_camera.gazebo.xacro (robot description, xacro)
@@ -14,5 +14,5 @@
       <updateRate>20.0</updateRate>
       <baseline>0.2</baseline>
-      <controller:gazebo_ros_camera name="${name}_depth_frame_controller" plugin="libgazebo_ros_camera.so">
+      <controller:gazebo_ros_camera name="${name}_depth_frame_controller" plugin="libgazebo_ros_openni_kinect.so">
         <alwaysOn>true</alwaysOn>
         <updateRate>20.0</updateRate>
@@ -39,7 +39,7 @@
       <updateRate>20.0</updateRate>
       <baseline>0.2</baseline>
-      <controller:gazebo_ros_camera name="${name}_rgb_frame_controller" plugin="libgazebo_ros_camera.so">
+      <controller:gazebo_ros_camera name="${name}_rgb_frame_controller" plugin="libgazebo_ros_openni_kinect.so">
         <alwaysOn>true</alwaysOn>
-        <updateRate>30.0</updateRate>
+        <updateRate>20.0</updateRate>
         <imageTopicName>/camera/rgb/image_raw</imageTopicName>
         <cameraInfoTopicName>/camera/rgb/camera_info</cameraInfoTopicName>

Commit message: better problem for tro

File: youbot_description/robots/youbot.urdf.xacro (robot description, xacro)
@@ -23,5 +23,4 @@
   <xacro:include filename="$(find youbot_description)/urdf/sensors/hokuyo_urg04_laser.urdf.xacro"/>
   <!-- kinect -->
-  <xacro:include filename="$(find youbot_description)/urdf/sensors/kinect_camera.urdf.xacro"/>
   <xacro:include filename="$(find common_sensors)/urdf/sensors/kinect2.urdf.xacro"/>
   <!-- Now we can start using the macros xacro:included above to define the actual youbot -->
@@ -50,5 +49,5 @@
   <!-- kinect2 camera from Jennifer Buehler -->
   <xacro:kinect2 name="kinect_camera_rgb" parent="base_link" >
-    <origin xyz="${0.35} 0 0.25" rpy="0 0 0" />
+    <origin xyz="${0.3} 0 0.18" rpy="0 0 0" />
   </xacro:kinect2>
 </robot>

Commit message: updated code

File: youbot_description/robots/youbot.urdf.xacro (robot description, xacro)
@@ -49,5 +49,5 @@
   <!-- kinect2 camera from Jennifer Buehler -->
   <xacro:kinect2 name="kinect_camera_rgb" parent="base_link" >
-    <origin xyz="${0.3} 0 0.18" rpy="0 0 0" />
+    <origin xyz="${0.4} 0 0.28" rpy="0 ${M_PI/18} 0" />
   </xacro:kinect2>
 </robot>

Commit message: reorganized dir structure

File: youbot_description/robots/youbot.urdf.xacro (robot description, xacro)
@@ -49,5 +49,5 @@
   <!-- kinect2 camera from Jennifer Buehler -->
   <xacro:kinect2 name="kinect_camera_rgb" parent="base_link" >
-    <origin xyz="${0.4} 0 0.28" rpy="0 ${M_PI/18} 0" />
+    <origin xyz="${0.4} 0 0.48" rpy="0 ${M_PI/20} 0" />
   </xacro:kinect2>
 </robot>

File: youbot_description/urdf/youbot_base/base.urdf.xacro (robot description, xacro)
@@ -55,5 +55,5 @@
     </link>
     <joint name="${name}_footprint_joint" type="fixed">
-      <origin xyz="${base_offset} 0 0" rpy="0 0 0"/>
+      <origin xyz="0 0 0" rpy="0 0 0"/>
       <child link="${name}_link"/>
       <parent link="${name}_footprint"/>

Commit message: designing visuomotor policy

File: youbot_description/robots/youbot.urdf.xacro (robot description, xacro)
@@ -24,4 +24,6 @@
   <!-- kinect -->
   <xacro:include filename="$(find common_sensors)/urdf/sensors/kinect2.urdf.xacro"/>
+  <!-- youbot obstacle -->
+  <!-- <xacro:include filename="$(find youbot_description)/urdf/youbot_obstacle/obstacle.urdf.xacro" /> -->
   <!-- Now we can start using the macros xacro:included above to define the actual youbot -->
   <!-- The first use of a macro.  This one was defined in base.urdf.xacro above.
@@ -49,5 +51,10 @@
   <!-- kinect2 camera from Jennifer Buehler -->
   <xacro:kinect2 name="kinect_camera_rgb" parent="base_link" >
-    <origin xyz="${0.4} 0 0.48" rpy="0 ${M_PI/20} 0" />
+    <origin xyz="${0.4} 0 0.42" rpy="0 ${M_PI/10} 0" />
   </xacro:kinect2>
+  <!-- World obstacle -->
+<!--   <xacro:youbot_obstacle name="youbot_obstacle" parent="youbot_obstacle_right_corner_wall" >
+    <origin xyz="${0.0} 0 0.0" rpy="0 ${0/10} 0" />
+  </xacro:youbot_obstacle> -->
+    <!-- <xacro:macro name="youbot_obstacle"> -->
 </robot>

File: youbot_description/urdf/youbot_base/base.urdf.xacro (robot description, xacro)
@@ -37,9 +37,9 @@
       <inertial>
         <mass value="0.1"/>
-        <origin xyz="0 0 ${-base_size_z / 2.0}" rpy="0 0 0"/>
+        <origin xyz="${base_offset} 0 ${-base_size_z / 2.0}" rpy="0 0 0"/>
         <inertia ixx="1.0" ixy="0.0" ixz="0.0" iyy="1.0" iyz="0.0" izz="1.0"/>
       </inertial>
       <visual>
-        <origin xyz="0 0 0" rpy="0 0 0"/>
+        <origin xyz="${base_offset} 0 0" rpy="0 0 0"/>
         <geometry>
           <box size="0.001 0.001 0.001"/>
@@ -48,5 +48,5 @@
       </visual>
       <collision>
-        <origin xyz="0 0 ${-base_size_z / 2.0}" rpy="0 0 0"/>
+        <origin xyz="${base_offset} 0 ${-base_size_z / 2.0}" rpy="0 0 0"/>
         <geometry>
           <box size="0.001 0.001 0.001"/>
@@ -55,5 +55,5 @@
     </link>
     <joint name="${name}_footprint_joint" type="fixed">
-      <origin xyz="0 0 0" rpy="0 0 0"/>
+      <origin xyz="${base_offset} 0 0" rpy="0 0 0"/>
       <child link="${name}_link"/>
       <parent link="${name}_footprint"/>

File: youbot_description/urdf/youbot_obstacle/obstacle.gazebo.xacro (robot description, xacro)
@@ -4,7 +4,10 @@
        xmlns:interface="http://playerstage.sourceforge.net/gazebo/xmlschema/#interface"
        xmlns:xacro="http://ros.org/wiki/xacro">
-  <xacro:macro name="youbot_obstacle_box_gazebo">
-    <gazebo reference="youbot_obstacle">
+  <xacro:macro name="youbot_obstacle_gazebo">
+    <gazebo reference="youbot_obstacle_box">
       <material value="Gazebo/Orange" />
+    </gazebo>
+    <gazebo reference="youbot_obstacle_right_corner_wall">
+      <material value="Gazebo/Gray" />
     </gazebo>
   </xacro:macro>

File: youbot_description/urdf/youbot_obstacle/obstacle.urdf.xacro (robot description, xacro)
@@ -4,7 +4,18 @@
        xmlns:interface="http://playerstage.sourceforge.net/gazebo/xmlschema/#interface"
        xmlns:xacro="http://ros.org/wiki/xacro">
-  <xacro:include filename="$(find youbot_description)/urdf/youbot_obstacle/obstacle.gazebo.xacro"/>
-  <xacro:macro name="youbot_obstacle" params="name">
-    <link name="${name}_box">
+  <xacro:property name="material_orange">
+    <material name="orange">
+      <color rgba="1.0 0.7 0.0 1"/>
+    </material>
+  </xacro:property>
+<!--   <xacro:include filename="$(find youbot_description)/urdf/youbot_obstacle/obstacle.gazebo.xacro"/> -->
+    <gazebo reference="youbot_obstacle_box">
+      <material value="Gazebo/Orange" />
+    </gazebo>
+<!--     <gazebo reference="youbot_obstacle_right_corner_wall">
+      <material value="Gazebo/Gray" />
+    </gazebo>   -->
+  <!-- <xacro:macro name="youbot_obstacle"> -->
+    <link name="youbot_obstacle_box">
       <inertial>
          <mass value="1e-2"/>
@@ -24,16 +35,35 @@
          <origin xyz="0 0 0" rpy="0 0 0" />
          <geometry>
-          <box size="${2*0.15748} ${2*0.15748} ${0.35*0.8508}}"  />
+          <box size="${2*0.15748} ${2*0.15748} ${0.35*0.8508}"  />
          </geometry>
+         <material name="orange"/>
       </collision>
     </link>
-    <!-- youbot obstacle -->
-    <joint name="${name}_joint" type="fixed">
-      <origin xyz="${5*0.6} -0.15 0.0" rpy="0 0 0"/>
-      <parent link="wall_8"/>
-      <child link="${name}_box"/>
-    </joint>
-    <!-- extensions -->
-    <xacro:obstacle_box_gazebo/>
-  </xacro:macro>
+ <!--    <link name="youbot_obstacle_right_corner_wall">
+      <inertial>
+        <origin xyz="0 0.0 -0.075" />
+        <mass value="10.0" />
+        <inertia  ixx="1.0" ixy="0.0"  ixz="0.0"  iyy="1.0"  iyz="0.0"  izz="1.0" />
+      </inertial>
+      <visual>
+        <origin xyz="0 0.0 -0.075"/>
+        <geometry>
+          <box size="0.5 0.8 0.15" />
+        </geometry>
+      </visual>
+      <collision>
+        <origin xyz="0 0.0 -0.075" />
+        <geometry>
+        <box size="0.5 0.8 0.15" />
+        </geometry>
+      </collision>
+    </link>
+    <joint name="youbot_obstacle_joint" type="fixed">
+      <origin xyz="${5*0.7} 0.15 0.0" rpy="0 0 0"/>
+      <parent link="youbot_obstacle_right_corner_wall"/>
+      <child link="youbot_obstacle_box"/>
+    </joint> -->
+    <!-- extensions --><!--
+    <xacro:youbot_obstacle_gazebo name="youbot_obstacle"/> -->
+  <!-- </xacro:macro> -->
 </robot>

File: youbot_simulation/youbot_gazebo_worlds/urdf/robocup_at_work_2012.urdf (robot description, URDF)
Before this commit: robot arena, 9 links, 8 joints
Links:
- removed link orange_box
Joints:
- removed joint join_box
