Commit message: large controls

File: youbot_description/urdf/youbot_base/base.urdf.xacro (robot description, xacro)
@@ -37,9 +37,9 @@
       <inertial>
         <mass value="0.1"/>
-        <origin xyz="${base_offset} 0 ${-base_size_z / 2.0}" rpy="0 0 0"/>
+        <origin xyz="0 0 ${-base_size_z / 2.0}" rpy="0 0 0"/>
         <inertia ixx="1.0" ixy="0.0" ixz="0.0" iyy="1.0" iyz="0.0" izz="1.0"/>
       </inertial>
       <visual>
-        <origin xyz="${base_offset} 0 0" rpy="0 0 0"/>
+        <origin xyz="0 0 0" rpy="0 0 0"/>
         <geometry>
           <box size="0.001 0.001 0.001"/>
@@ -48,5 +48,5 @@
       </visual>
       <collision>
-        <origin xyz="${base_offset} 0 ${-base_size_z / 2.0}" rpy="0 0 0"/>
+        <origin xyz="0 0 ${-base_size_z / 2.0}" rpy="0 0 0"/>
         <geometry>
           <box size="0.001 0.001 0.001"/>
@@ -55,5 +55,5 @@
     </link>
     <joint name="${name}_footprint_joint" type="fixed">
-      <origin xyz="${base_offset} 0 0" rpy="0 0 0"/>
+      <origin xyz="0 0 0" rpy="0 0 0"/>
       <child link="${name}_link"/>
       <parent link="${name}_footprint"/>
